Commit message: feat: integrate web dashboard telemetry, fps tracking, and camera noise

File: model/robot.xacro (robot description, xacro)
@@ -181,4 +181,53 @@
             <joint_name>left_wheel_joint</joint_name>
         </plugin>
+        <plugin filename="gz-sim-sensors-system" name="gz::sim::systems::Sensors">
+            <render_engine>ogre</render_engine>
+        </plugin>
+    </gazebo>
+    <!-- Camera -->
+    <link name="camera_link">
+        <visual>
+            <origin xyz="0 0 0" rpy="0 0 0"/>
+            <geometry>
+                <box size="0.05 0.05 0.05"/>
+            </geometry>
+            <material name="camera_mat">
+                <color rgba="0 0 1 1"/>
+            </material>
+        </visual>
+    </link>
+    <joint name="camera_joint" type="fixed">
+        <origin xyz="${body_length/2} 0 ${body_height}" rpy="0 0 0"/>
+        <parent link="body_link"/>
+        <child link="camera_link"/>
+    </joint>
+    <gazebo reference="camera_link">
+        <sensor name="camera_sensor" type="camera">
+            <pose>0 0 0 0 0 0</pose>
+            <visualize>true</visualize>
+            <update_rate>30.0</update_rate>
+            <camera>
+                <horizontal_fov>0.9599</horizontal_fov>
+                <image>
+                    <width>1280</width>
+                    <height>720</height>
+                    <format>R8G8B8</format>
+                </image>
+                <clip>
+                    <near>0.1</near>
+                    <far>100</far>
+                </clip>
+                <noise>
+                    <type>gaussian</type>
+                    <mean>0.0</mean>
+                    <stddev>0.005</stddev>
+                </noise>
+            </camera>
+            <topic>camera/image_raw</topic>
+        </sensor>
+        <plugin filename="gz-sim-image-publisher-system" name="gz::sim::systems::ImagePublisher">
+            <topic>camera/image_raw/compressed</topic>
+            <format>JPG</format>
+        </plugin>
     </gazebo>
 </robot>
